File: SEPIC_CAD.kicad_sch (KiCad schematic)
At the start: 25 parts, among them IC1 LM5155DSSR, Q1 CSD18537NQ5A

Commit message: Look on my works ye mighty
Parts:
- removed C1, C2, C4: 10u, symbol Device:C
- removed C10, C3: 100p, symbol Device:C
- removed C11: 9.4u, symbol Device:C
- removed C12: 66u, symbol Device:C
- removed C5: 270p, symbol Device:C
- removed C6: 100n, symbol Device:C
- removed C7: 220n, symbol Device:C
- removed C8: 6.8n, symbol Device:C
- removed C9: 1u, symbol Device:C
- removed D1: STPS20M100SG-TR, D2PAK_STM, symbol 2022-11-06_22-07-15:STPS20M100SG-TR
- removed IC1: LM5155DSSR, SON50P200X300X80-13N-D, symbol Global Symbols:LM5155DSSR
- removed L1: 7448700015, symbol Device:L_Coupled
- removed Q1: CSD18537NQ5A, CSD19531Q5AT, symbol SamacSys_Parts:CSD18537NQ5A
- removed R1: 6k8, symbol Device:R_US
- removed R2: 34k8, symbol Device:R_US
- removed R3: 17k8, symbol Device:R_US
- removed R4: 10k, symbol Device:R_US
- removed R5: 100, symbol Device:R_US
- removed R6, R7: 4m, symbol Device:R_US
- removed R8: 51k1, symbol Device:R_US
- removed R9: 4k7, symbol Device:R_US
- added C?: 9.4u, symbol Device:C
- added C?: 220n, symbol Device:C
- added C?: 6.8n, symbol Device:C
- added C? (x2): 100p, symbol Device:C
- added C? (x3): 10u, symbol Device:C
- added C?: 270p, symbol Device:C
- added C?: 1u, symbol Device:C
- added C?: 66u, symbol Device:C
- added C?: 100n, symbol Device:C
- added D?: STPS20M100SG-TR, D2PAK_STM, symbol Global Symbols:STPS20M100SG-TR
- added IC?: LM5155DSSR, SON50P200X300X80-13N-D, symbol Global Symbols:LM5155DSSR
- added L?: 7448700015, symbol Device:L_Coupled
- added Q?: CSD18537NQ5A, CSD19531Q5AT, symbol Global Symbols:CSD18537NQ5A
- added R?: 17k8, symbol Device:R_US
- added R?: 4k7, symbol Device:R_US
- added R?: 34k8, symbol Device:R_US
- added R? (x2): 4m, symbol Device:R_US
- added R?: 100, symbol Device:R_US
- added R?: 51k1, symbol Device:R_US
- added R?: 10k, symbol Device:R_US
- added R?: 6k8, symbol Device:R_US
Connections:
- net 12V_Reg: now also C?.1, D?.3, R?.1
- net COMP: now also C?.1, C?.1, IC?.6 (COMP)
- net FB: now also IC?.8 (FB), R?.1, R?.2
- net GND: now also C?.1, C?.1, C?.2, C?.2, C?.2, C?.2, C?.2, C?.2, C?.2, C?.2, IC?.13 (EP), IC?.4 (PGND), IC?.7 (AGND), L?.3, R?.1, R?.2, R?.2, R?.2, R?.2
- net RT: now also IC?.10 (RT), R?.2
- net SS: now also C?.1, IC?.9 (SS)
- net UVLO: now also C?.1, IC?.12 (UVLO/SYNC), R?.1, R?.2
- net Vin: now also C?.1, C?.1, C?.1, C?.1, IC?.1 (BIAS), L?.1, R?.1
- new net: Q?.1 (S_1), Q?.2 (S_2), Q?.3 (S_3), R?.1, R?.1
- new net: IC?.3 (GATE), Q?.4 (G)
- new net: C?.2, L?.2, Q?.5 (D_1), Q?.6 (D_2), Q?.7 (D_3), Q?.8 (D_4)
- new net: C?.1, D?.1, L?.4
- new net: R?.1, R?.2
- new net: C?.2, R?.1
- new net: C?.2, IC?.5 (CS), R?.2
- new net: C?.2, IC?.2 (VCC)
Other:
- note added: "Design based on this \/"
- note added: "https://www.ti.com/lit/ug/snvu628/snvu628.pdf?ts=1667746686718"

Commit message: small tweaks
Parts:
- gave numbers to parts that had none: 25
Other:
- moved on the sheet: C11
